Commit message: Add CUDA-backed navigation observation and reorganize documentation
Add RGB-D capture, local visual question answering, and guarded navigation-observation tasks. Introduce a standalone CUDA model service with startup and in-navigation preloading, AMCL startup priors, velocity routing fixes, regression tests, and workflow-oriented documentation.

File: wheel_arm_description/urdf/wheel_arm.urdf.xacro (robot description, xacro)
@@ -316,4 +316,11 @@
     <origin xyz="0.34 0 ${base_height - 0.04}" rpy="0 0 0"/>
   </joint>
+  <!-- Optical coordinates: x right, y down, z forward. -->
+  <link name="camera_optical_frame"/>
+  <joint name="camera_optical_joint" type="fixed">
+    <parent link="camera_link"/>
+    <child link="camera_optical_frame"/>
+    <origin xyz="0 0 0" rpy="${-pi/2} 0 ${-pi/2}"/>
+  </joint>
   <gazebo reference="base_link">
     <material>Gazebo/DarkGrey</material>
@@ -371,7 +378,7 @@
   </gazebo>
   <gazebo reference="camera_link">
-    <sensor name="rgb_camera" type="camera">
-      <topic>/camera/image</topic>
-      <update_rate>30</update_rate>
+    <sensor name="rgbd_camera" type="rgbd_camera">
+      <topic>/camera</topic>
+      <update_rate>15</update_rate>
       <camera>
         <horizontal_fov>1.047</horizontal_fov>
@@ -382,6 +389,6 @@
         </image>
         <clip>
-          <near>0.05</near>
-          <far>20.0</far>
+          <near>0.1</near>
+          <far>8.0</far>
         </clip>
       </camera>
